File: pcb/xbee-adapter.kicad_sch (KiCad schematic)
At the start: 12 parts, among them J1 MCU, J2 Indicator, M1 DIGI_XBEE

Commit message: Adds resistors for the indicator LEDs
Parts:
- added R1, R2: 270Ω, Resistor_SMD:R_0805_2012Metric, symbol Device:R
Connections:
- net ASSOCIATE: now also R1.2; no longer M1.15 (Associate/DIO5/AD5)
- net ON/SLEEP: now also R2.2; no longer M1.13 (ON/SLEEP)
- new net: M1.15 (Associate/DIO5/AD5), R1.1
- new net: M1.13 (ON/SLEEP), R2.1
Other:
- title: LPS XBee Adapter LPS-X-1 -> LPS-X-1 Leawood Power Sensor XBee Adapter 1.
Changed lines of the file:
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@@
   (paper "A4")
   (title_block
-    (title "LPS XBee Adapter LPS-X-1")
-    (date "2024-01-28")
-    (rev "1.0")
+    (title "LPS-X-1 Leawood Power Sensor XBee Adapter 1.")
+    (date "2024-01-30")
+    (rev "1.1")
   )
   (junction (at 139.7 45.72) (diameter 0) (color 0 0 0 0)
@@
     (stroke (width 0) (type default))
   )
-  (wire (pts (xy 173.99 81.28) (xy 191.77 81.28))
+  (wire (pts (xy 173.99 81.28) (xy 177.8 81.28))
     (stroke (width 0) (type default))
   )
@@
     (stroke (width 0) (type default))
   )
-  (wire (pts (xy 173.99 86.36) (xy 191.77 86.36))
+  (wire (pts (xy 173.99 86.36) (xy 177.8 86.36))
+    (stroke (width 0) (type default))
+  )
+  (wire (pts (xy 185.42 81.28) (xy 198.12 81.28))
     (stroke (width 0) (type default))
   )
@@
   )
   (wire (pts (xy 100.33 73.66) (xy 118.11 73.66))
+    (stroke (width 0) (type default))
+  )
+  (wire (pts (xy 185.42 86.36) (xy 198.12 86.36))
     (stroke (width 0) (type default))
   )
@@
     (effects (font (size 1.27 1.27)) (justify left bottom))
   )
-  (label "ON{slash}SLEEP" (at 191.77 86.36 180) (fields_autoplaced)
+  (label "ON{slash}SLEEP" (at 198.12 86.36 180) (fields_autoplaced)
     (effects (font (size 1.27 1.27)) (justify right bottom))
   )
@@
     (effects (font (size 1.27 1.27)) (justify right bottom))
   )
-  (label "ASSOCIATE" (at 191.77 81.28 180) (fields_autoplaced)
+  (label "ASSOCIATE" (at 198.12 81.28 180) (fields_autoplaced)
     (effects (font (size 1.27 1.27)) (justify right bottom))
   )
@@
         (path "/3c8aa795-42f1-4d19-a1e9-ad92c16c05d6"
           (reference "H4") (unit 1)
+        )
+      )
+    )
+  )
+  (symbol (lib_id "Device:R") (at 181.61 81.28 90) (unit 1)
+    (in_bom yes) (on_board yes) (dnp no) (fields_autoplaced)
+    (property "Reference" "R1" (at 181.61 76.1197 90)
+      (effects (font (size 1.27 1.27)))
+    )
+    (property "Value" "270Ω" (at 181.61 78.5439 90)
+      (effects (font (size 1.27 1.27)))
+    )
+    (property "Footprint" "Resistor_SMD:R_0805_2012Metric" (at 181.61 83.058 90)
+      (effects (font (size 1.27 1.27)) hide)
+    )
+    (property "Datasheet" "~" (at 181.61 81.28 0)
+      (effects (font (size 1.27 1.27)) hide)
+    )
+    (pin "1")
+    (pin "2")
+    (instances
+      (project "xbee-adapter"
+        (path "/3c8aa795-42f1-4d19-a1e9-ad92c16c05d6"
+          (reference "R1") (unit 1)
         )
       )
@@
     )
     (property "Footprint" "XBee-Adapter:XBEE_S2C" (at 129.54 82.55 0)
-      (effects (font (size 1.524 1.524)))
+      (effects (font (size 1.524 1.524)) hide)
     )
     (property "Datasheet" "" (at 129.54 82.55 0)
@@
         )
       )
+    )
+  )
+  (symbol (lib_id "Device:R") (at 181.61 86.36 90) (unit 1)
+    (in_bom yes) (on_board yes) (dnp no)
+    (property "Reference" "R2" (at 181.61 88.9 90)
+      (effects (font (size 1.27 1.27)))
+    )
+    (property "Value" "270Ω" (at 181.61 91.44 90)
+      (effects (font (size 1.27 1.27)))
+    )
+    (property "Footprint" "Resistor_SMD:R_0805_2012Metric" (at 181.61 88.138 90)
+      (effects (font (size 1.27 1.27)) hide)
+    )
+    (property "Datasheet" "~" (at 181.61 86.36 0)
+      (effects (font (size 1.27 1.27)) hide)
+    )
+    (pin "1")
+    (pin "2")
+    (instances
+      (project "xbee-adapter"
+        (path "/3c8aa795-42f1-4d19-a1e9-ad92c16c05d6"
+          (reference "R2") (unit 1)
+        )
+      )

Commit message: Adds a ground pin for the inticator connector
Parts:
- removed J2: Indicator, Connector_PinHeader_2.54mm:PinHeader_1x02_P2.54mm_Vertical, symbol Connector:Conn_01x02_Pin
- added J2: Indicator, Connector_PinHeader_2.54mm:PinHeader_1x03_P2.54mm_Vertical, symbol Connector:Conn_01x03_Pin
Connections:
- net ASSOCIATE: now also J2.1 (Pin_1)
- net GND: now also J2.3 (Pin_3)
- net ON/SLEEP: now also J2.2 (Pin_2)
